File: Circular_RPi5.kicad_sch (KiCad schematic)
At the start: 9 parts, among them J1 USB3_A, J2 Conn_01x22, J3 RJ45_LED, J4 USB_C_Receptacle_PowerOnly_6P, J5 HDMI_D_1.4, J6 Conn_02x20_Odd_Even

Commit message: LED fixed
Parts:
- added D1: LED, LED_SMD:LED_0603_1608Metric, symbol Device:LED
- added R3: 330 ohm, symbol Device:R
- added V1: 5, symbol Simulation_SPICE:VDC
Connections:
- net +5V: now also R3.1, V1.1
- net GND: now also D1.1 (K), V1.2
- new net: D1.2 (A), R3.2

Commit message: PCB Fixed
Parts:
- removed J3: RJ45_LED, Connector_RJ:RJ45_Molex_0855135013_Vertical, symbol Connector:RJ45_LED
- removed J6: Conn_02x20_Odd_Even, Connector_PinHeader_2.54mm:PinHeader_2x20_P2.54mm_Vertical, symbol Connector_Generic:Conn_02x20_Odd_Even
- removed V1: 5, symbol Simulation_SPICE:VDC
- added C1: 470uF, Capacitor_SMD:CP_Elec_8x10, symbol Device:C_Polarized
- added C2: 10uF, Capacitor_SMD:C_0805_2012Metric, symbol Device:C
- added C3, C4, C5, C6, C7, C8: 0.1uF, Capacitor_SMD:C_0805_2012Metric, symbol Device:C
- added D2: D_TVS, Diode_SMD:D_SMA, symbol Device:D_TVS
- added F1, F2: Polyfuse, Fuse:Fuse_1812_4532Metric, symbol Device:Polyfuse
- added J3: Conn_01x05, Connector_PinHeader_2.54mm:PinHeader_1x05_P2.54mm_Vertical, symbol Connector_Generic:Conn_01x05
- added J7: RJ45_Amphenol_RJMG1BD3B8K1ANR, Connector_RJ:RJ45_Amphenol_RJMG1BD3B8K1ANR, symbol Connector:RJ45_Amphenol_RJMG1BD3B8K1ANR
- added R4: 47k ohm, Resistor_SMD:R_0805_2012Metric, symbol Device:R
- added U1, U2, U3, U4, U5: USBLC6-2SC6, Package_TO_SOT_SMD:SOT-23-6, symbol Power_Protection:USBLC6-2SC6
- added U6: TPD4E05U06DQA, Package_SON:USON-10_2.5x1.0mm_P0.5mm, symbol Power_Protection:TPD4E05U06DQA
- added U7: TPS2069CDBV, Package_TO_SOT_SMD:SOT-23-5, symbol Power_Management:TPS2069CDBV
- added U8: USBLC6-4SC6, Package_TO_SOT_SMD:SOT-23-6, symbol Power_Protection:USBLC6-4SC6
- R3: footprint (none) -> Resistor_SMD:R_0805_2012Metric
Connections:
- net +3.3V: now also J3.1 (Pin_1)
- net +5V: now also C1.1, C2.1, C3.2, C4.1, C5.1, C6.1, C7.1, C8.1, D2.2 (A2), F1.2, F2.1, J3.5 (Pin_5), U1.5 (VBUS), U2.5 (VBUS), U3.5 (VBUS), U4.5 (VBUS), U5.5 (VBUS), U7.5 (IN); no longer J1.1 (VBUS), J4.A9 (VBUS), J4.B9 (VBUS), J5.19 (+5V)
- net GND: now also C1.2, C2.2, C3.1, C4.2, C5.2, C6.2, C7.2, C8.2, D2.1 (A1), J3.4 (Pin_4), J7.R8, J7.SH, R4.2, U1.2 (GND), U2.2 (GND), U3.2 (GND), U4.2 (GND), U5.2 (GND), U6.3 (GND), U6.8 (GND), U7.2 (GND), U8.2 (GND)
- net GPIO2: now also J3.2 (Pin_2)
- net GPIO3: now also J3.3 (Pin_3)
- net HDMI0_CLK_N: now also U5.3 (I/O2)
- net HDMI0_CLK_P: now also U5.1 (I/O1)
- net HDMI0_HOTPLUG: now also R4.1
- net HDMI0_TX0_N: now also U4.3 (I/O2)
- net HDMI0_TX0_P: now also U4.1 (I/O1)
- net HDMI0_TX1_N: now also U3.3 (I/O2)
- net HDMI0_TX1_P: now also U3.1 (I/O1)
- net HDMI0_TX2_N: now also U2.3 (I/O2)
- net HDMI0_TX2_P: now also U2.1 (I/O1)
- net at J1.2 (D-), Module1.103 (USB2_N): now also U1.1 (I/O1)
- net at J1.3 (D+), Module1.105 (USB2_P): now also U1.3 (I/O2)
- net SSRX-: now reaches J1.5 (SSRX-), Module1.128 (USB3-0-RX_N)
- net SSRX-: now also U6.5 (D2-)
- net SSRX+: now reaches J1.6 (SSRX+), Module1.130 (USB3-0-RX_P)
- net SSRX+: now also U6.4 (D2+)
- net SSTX-: now reaches J1.8 (SSTX-), Module1.140 (USB3-0-TX_N)
- net SSTX-: now also U6.2 (D1-)
- net SSTX+: now reaches J1.9 (SSTX+), Module1.142 (USB3-0-TX_P)
- net SSTX+: now also U6.1 (D1+)
- net Ethernet_Pair0_N: now reaches Module1.10 (Ethernet_Pair0_N)
- net Ethernet_Pair0_N: now also J7.R2 (TD-)
- net Ethernet_Pair0_P: now reaches Module1.12 (Ethernet_Pair0_P)
- net Ethernet_Pair0_P: now also J7.R1 (TD+)
- net Ethernet_Pair1_P: now reaches Module1.4 (Ethernet_Pair1_P)
- net Ethernet_Pair1_P: now also J7.R3 (RD+)
- net Ethernet_Pair1_N: now reaches Module1.6 (Ethernet_Pair1_N)
- net Ethernet_Pair1_N: now also J7.R6 (RD-)
- net VBUS_EN: now reaches Module1.111 (VBUS_EN)
- net VBUS_EN: now also U7.4 (EN)
- new net: J1.1 (VBUS), U7.1 (OUT)
- new net: F2.2, J5.19 (+5V)
- new net +3,3V: U8.5 (VBUS)
- new net MIPI_D0_N: U8.3 (I/O2)
- new net MIPI_D0_P: U8.1 (I/O1)
- new net MIPI_D1_N: U8.6 (I/O4)
- new net MIPI_D1_P: U8.4 (I/O3)
- new net VBUS_IN: F1.1, J4.A9 (VBUS), J4.B9 (VBUS)
- no-connect marks 0 -> 7
Other:
- moved on the sheet: D1, J1, J2, J4, J5, Module1A, Module1B, R1, R2, R3
