File: Circular_RPi5.kicad_sch (KiCad schematic)
At the start: 31 parts, among them J1 USB3_A, J2 Conn_01x22, J3 Conn_01x05, J4 USB_C_Receptacle_PowerOnly_6P, J5 HDMI_D_1.4, J7 RJ45_Amphenol_RJMG1BD3B8K1ANR, U1 USBLC6-2SC6, U2 USBLC6-2SC6, U3 USBLC6-2SC6, U4 USBLC6-2SC6, U5 USBLC6-2SC6, U6 TPD4E05U06DQA, U7 TPS2069CDBV, U8 USBLC6-4SC6

Commit message: Fix CM5 carrier board pre-fab issues: GPIO_VREF, USB3 D+/D-, MIPI ESD, Gigabit Ethernet, fuse rating
Schematic:
- Wire GPIO_VREF (CM5 pin 78) to +3.3V; the module datasheet requires this
  tied to CM5_3.3V or CM5_1.8V or the GPIO bank is unreferenced.
- Rewire J1's USB3 D+/D- from CM5 pins 105/103 (an unrelated standalone USB2
  port) to pins 134/136 (USB3-0-DP/DM), the correct companion pins for the
  SuperSpeed TX/RX lines already wired to that port.
- Fix U8 (USBLC6-4SC6) label typos: MIPI_D0/D1_* -> MIPI0_D0/D1_* and
  +3,3V -> +3.3V. U8 was sitting electrically isolated on orphan nets and
  provided no ESD protection on the MIPI0 camera lines.
- Replace J7 (Amphenol RJMG1BD3B8K1ANR, confirmed 10/100-only) with the UDE
  RB1-125B8G1A, a genuine 10/100/1000 magjack, and wire all 4 differential
  pairs plus its second ground pin.
- F1/F2: specify a real 5A/16V PTC (Littelfuse 2920L500/16MR) to meet the
  5V/5A input requirement; update footprints to Fuse_2920_7451Metric.

PCB:
- Relocate F1, F2, and R1 off the board edge (the 2920 footprint collided
  with the board outline and R1 at their original spots) to open,
  DRC-verified locations found via clearance search over actual pad/track/
  via geometry; F1/F2 footprints swapped to Fuse_2920_7451Metric to match.
- Swap J7 footprint to RJ45_UDE_RB1-125B8G1A; clean up all now-invalid
  copper from the swap and refill zones so the new through-hole pattern is
  properly cleared.
- Reassign pad nets throughout to match the schematic fixes above (GPIO_VREF,
  USB3 D+/D-, U8's MIPI/3.3V pins, J7's 8 differential pairs).

DRC is clean except for 22 documented ratsnest gaps (short local runs into
the CM5 module's 0.4mm-pitch connector field, plus the U8-to-J2/Module1 MIPI
splice) and one pre-existing SSTX+/SSTX- clearance graze against J7's SH pad
that three independent nudge attempts couldn't resolve without trading it for
a new violation elsewhere -- both need KiCad's interactive router to finish.

Co-Authored-By: Claude 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
Parts:
- removed J7: RJ45_Amphenol_RJMG1BD3B8K1ANR, Connector_RJ:RJ45_Amphenol_RJMG1BD3B8K1ANR, symbol Connector:RJ45_Amphenol_RJMG1BD3B8K1ANR
- added J7: RJ45_RB1-125B8G1A, Connector_RJ:RJ45_UDE_RB1-125B8G1A, symbol Connector:RJ45_RB1-125B8G1A
- F1, F2: value Polyfuse -> 2920L500/16MR; footprint Fuse:Fuse_1812_4532Metric -> Fuse:Fuse_2920_7451Metric
Connections:
- net +3,3V is gone; now on net +3.3V: U8.5 (VBUS)
- net MIPI_D0_N is gone; now on net MIPI0_D0_N: U8.3 (I/O2)
- net MIPI_D0_P is gone; now on net MIPI0_D0_P: U8.1 (I/O1)
- net MIPI_D1_N is gone; now on net MIPI0_D1_N: U8.6 (I/O4)
- net MIPI_D1_P is gone; now on net MIPI0_D1_P: U8.4 (I/O3)
- net +3.3V: now also Module1.78 (GPIO_VREF(1.8v/3.3v_Input))
- net Ethernet_Pair0_N: now also J7.R3 (TD1-)
- net Ethernet_Pair0_P: now also J7.R2 (TD1+)
- net Ethernet_Pair1_N: now also J7.R5 (TD2-)
- net Ethernet_Pair1_P: now also J7.R4 (TD2+)
- net GND: now also J7.R10 (GND), J7.SH
- net USB3-0-D_N: now reaches J1.2 (D-), U1.1 (I/O1)
- net USB3-0-D_N: now also Module1.136 (USB3-0-D_N); no longer Module1.103 (USB2_N)
- net USB3-0-D_P: now reaches J1.3 (D+), U1.3 (I/O2)
- net USB3-0-D_P: now also Module1.134 (USB3-0-D_P); no longer Module1.105 (USB2_P)
- net Ethernet_Pair2_P: now reaches Module1.11 (Ethernet_Pair2_P)
- net Ethernet_Pair2_P: now also J7.R6 (TD3+)
- net Ethernet_Pair3_P: now reaches Module1.3 (Ethernet_Pair3_P)
- net Ethernet_Pair3_P: now also J7.R8 (TD4+)
- net Ethernet_Pair3_N: now reaches Module1.5 (Ethernet_Pair3_N)
- net Ethernet_Pair3_N: now also J7.R9 (TD4-)
- net Ethernet_Pair2_N: now reaches Module1.9 (Ethernet_Pair2_N)
- net Ethernet_Pair2_N: now also J7.R7 (TD3-)
- no-connect marks 7 -> 2

Commit message: Rebuild J4 5V power entry as copper zones; scope custom DRC rules correctly
DRC IS NOT CLEAN after this commit -- 201 violations remain and they are real.
See the breakdown at the end of this message. This commit is an improvement to
the J4 power entry, not a release gate.

J4 VBUS_IN power entry rebuilt:
- Deleted 19.2mm of 0.25mm-wide VBUS_IN track snaking around J4. On 1oz outer
  copper that carries ~0.88A; it was being asked to carry 5A, so it was acting
  as a fuse. The pre-existing 2.8mm trunk out to F1 was left intact.
- Added two VBUS_IN copper zones: F.Cu 26.25 mm2 (left pocket plus a corridor
  north to the existing trunk via at 105.2,97.8) and B.Cu 58.68 mm2 (under the
  connector, north to the trunk). Both use solid pad connection -- thermal
  spokes would choke 5A.
- Added 7 vias at 0.8mm dia / 0.4mm drill: two bridging the A/B pad rows
  (106.562,89.086 and 106.750,93.000) and five stitching top-to-bottom in the
  left corridor at x=102.6. Every position was validated against pads, tracks,
  vias, board edge and the J4/J5 footprint keepouts on both outer layers before
  placement.
- Added two 0.5mm neck-down stubs from B4 and B9 into their bridge vias. B4 was
  otherwise held by only a 0.14mm via-annulus overlap, worth ~1.16A against a
  ~1.25A per-pin share.

Measured result: narrowest neck is F.Cu 0.76mm in parallel with B.Cu 3.14mm,
about 8.6A at a 10C rise -- comfortably over the 5A requirement. All four VBUS
pads (A4, A9, B4, B9) confirmed connected; 0 unconnected items. This rebuild
added zero DRC violations.

The requested 0.6mm vias immediately right of B4/B9, and 0.5mm tracks left out
of A4/A9, are both geometrically impossible: the S1 shield pads (PTH, 1.1mm,
all layers) sit directly left of A4/A9 and directly right of B4/B9, leaving
only a 0.34mm gap. The inter-row channel was used instead.

Custom DRC rules corrected -- two genuine flaws in rules I wrote earlier:
- 5A power minimum lowered 3.0mm -> 2.5mm. IPC-2221 on this stackup's 1oz
  o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
Parts:
- added C9: 22uF, Capacitor_SMD:C_1206_3216Metric, symbol Device:C
- J1: footprint Connector_USB:USB_A_Molex_105057_Vertical -> Connector_USB:USB3_A_Molex_48393-001
Connections:
- net GND: now also J1.7 (DRAIN), C9.2
- net at J1.1 (VBUS), U7.1 (OUT): now also C9.1
Changed lines of the file:
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@@
 	(wire
 		(pts
-			(xy 69.85 102.87) (xy 74.93 102.87)
+			(xy 69.85 102.87) (xy 72.39 102.87)
 		)
 		(stroke
@@
 	(wire
 		(pts
-			(xy 87.63 57.15) (xy 87.63 69.85)
+			(xy 87.63 57.15) (xy 87.63 63.5)
 		)
 		(stroke
@@
 		)
 	)
+	(wire
+		(pts
+			(xy 87.63 63.5) (xy 93.98 63.5)
+		)
+		(stroke
+			(width 0)
+			(type default)
+		)
+	)
+	(junction
+		(at 87.63 63.5)
+		(diameter 0)
+		(color 0 0 0 0)
+	)
+	(symbol
+		(lib_id "Device:C")
+		(at 93.98 67.31 0)
+		(unit 1)
+		(exclude_from_sim no)
+		(in_bom yes)
+		(on_board yes)
+		(dnp no)
+		(fields_autoplaced yes)
+		(property "Reference" "C9"
+			(at 97.79 66.0399 0)
+			(effects
+				(font
+					(size 1.27 1.27)
+				)
+				(justify left)
+			)
+		)
+		(property "Value" "22uF"
+			(at 97.79 68.5799 0)
+			(effects
+				(font
+					(size 1.27 1.27)
+				)
+				(justify left)
+			)
+		)
+		(property "Footprint" "Capacitor_SMD:C_1206_3216Metric"
+			(at 94.9452 71.12 0)
+			(effects
+				(font
+					(size 1.27 1.27)
+				)
+				(hide yes)
+			)
+		)
+		(property "Datasheet" "~"
+			(at 93.98 67.31 0)
+			(effects
+				(font
+					(size 1.27 1.27)
+				)
+				(hide yes)
+			)
+		)
+		(property "Description" "USB VBUS bulk / TPS2069 output stability capacitor"
+			(at 93.98 67.31 0)
+			(effects
+				(font
+					(size 1.27 1.27)
+				)
+				(hide yes)
+			)
+		)
+		(pin "1"
+		)
+		(pin "2"
+		)
+		(instances
+			(project ""
+				(path "/f9e30a80-9e2f-4005-8ba2-00bc0bf441f1"
+					(reference "C9")
+					(unit 1)
+				)
+			)
+		)
+	)
+	(symbol
+		(lib_id "power:GND")
+		(at 93.98 71.12 0)
+		(unit 1)
+		(exclude_from_sim no)
+		(in_bom yes)
+		(on_board yes)
+		(dnp no)
+		(fields_autoplaced yes)
+		(property "Reference" "#PWR0104"
+			(at 93.98 77.47 0)
+			(effects
+				(font
+					(size 1.27 1.27)
+				)
+				(hide yes)
+			)
+		)
+		(property "Value" "GND"
+			(at 93.98 76.2 0)
+			(effects
+				(font
+					(size 1.27 1.27)
+				)
+			)
+		)
+		(property "Footprint" ""
+			(at 93.98 71.12 0)
+			(effects
+				(font
+					(size 1.27 1.27)
+				)
+				(hide yes)
+			)
+		)
+		(property "Datasheet" ""
+			(at 93.98 71.12 0)
+			(effects
+				(font
+					(size 1.27 1.27)
+				)
+				(hide yes)
+			)
+		)
+		(property "Description" "Power symbol creates a global label with name \"GND\" , ground"
+			(at 93.98 71.12 0)
+			(effects
+				(font
+					(size 1.27 1.27)
+				)
+				(hide yes)
+			)
+		)
+		(pin "1"
+		)
+		(instances
+			(project ""
+				(path "/f9e30a80-9e2f-4005-8ba2-00bc0bf441f1"
+					(reference "#PWR0104")
+					(unit 1)
+				)
+			)
+		)
+	)
+	(wire
+		(pts
+			(xy 87.63 63.5) (xy 87.63 69.85)
+		)
+		(stroke
+			(width 0)
+			(type default)
+		)
+	)
+	(wire
+		(pts
+			(xy 72.39 102.87) (xy 74.93 102.87)
+		)
+		(stroke
+			(width 0)
+			(type default)
+		)
+	)
+	(wire
+		(pts
+			(xy 72.39 97.79) (xy 72.39 102.87)
+		)
+		(stroke
+			(width 0)
+			(type default)
+		)
+	)
+	(junction
+		(at 72.39 102.87)
+		(diameter 0)
+		(color 0 0 0 0)
+	)
 	(symbol
 		(lib_id "Connector:USB3_A")
@@
 			)
 		)
-		(property "Footprint" "Connector_USB:USB_A_Molex_105057_Vertical"
+		(property "Footprint" "Connector_USB:USB3_A_Molex_48393-001"
 			(at 78.74 77.47 0)
 			(effects
