File: Circular_RPi5.kicad_pcb (KiCad board)
At the start: 8 copper layers, 80 x 80 mm, 11 parts, among them J1 USB3_A, J2 Conn_01x22, J3 RJ45_LED, J4 USB_C, J5 HDMI_D_1.4, J6 GPIO PINS

Commit message: LED fixed
Parts:
- REF**: value R_LED -> 330 ohm
- turned REF** to 0 degrees
Connections:
- REF** pad 1: LED_LOOP -> GND
- REF** pad 2: GND -> LED_LOOP
Changed lines of the file:
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@@
 		(locked yes)
 		(layer "B.Cu")
-		(at 158.496 128.016 180)
+		(at 158.496 128.016)
 		(descr "LED SMD 0603 (1608 Metric), square (rectangular) end terminal, IPC-7351 nominal, (Body size source: http://www.tortai-tech.com/upload/download/2011102023233369053.pdf), generated with kicad-footprint-generator")
 		(tags "LED")
@@
 		)
 		(property "Value" "LED_P"
-			(at 0 -1.43 0)
+			(at 0.254 1.524 0)
 			(layer "B.Fab")
 			(effects
@@
 		)
 		(attr smd)
+		(fp_line
+			(start -1.485 -0.735)
+			(end 0.8 -0.735)
+			(stroke
+				(width 0.12)
+				(type solid)
+			)
+			(layer "B.SilkS")
+		)
+		(fp_line
+			(start -1.485 0.735)
+			(end -1.485 -0.735)
+			(stroke
+				(width 0.12)
+				(type solid)
+			)
+			(layer "B.SilkS")
+		)
 		(fp_line
 			(start 0.8 0.735)
@@
 		)
 		(fp_line
-			(start -1.485 0.735)
-			(end -1.485 -0.735)
-			(stroke
-				(width 0.12)
-				(type solid)
-			)
-			(layer "B.SilkS")
-		)
-		(fp_line
-			(start -1.485 -0.735)
-			(end 0.8 -0.735)
-			(stroke
-				(width 0.12)
-				(type solid)
-			)
-			(layer "B.SilkS")
+			(start -1.48 -0.73)
+			(end -1.48 0.73)
+			(stroke
+				(width 0.05)
+				(type solid)
+			)
+			(layer "B.CrtYd")
+		)
+		(fp_line
+			(start -1.48 0.73)
+			(end 1.48 0.73)
+			(stroke
+				(width 0.05)
+				(type solid)
+			)
+			(layer "B.CrtYd")
+		)
+		(fp_line
+			(start 1.48 -0.73)
+			(end -1.48 -0.73)
+			(stroke
+				(width 0.05)
+				(type solid)
+			)
+			(layer "B.CrtYd")
 		)
 		(fp_line
@@
 		)
 		(fp_line
-			(start 1.48 -0.73)
-			(end -1.48 -0.73)
-			(stroke
-				(width 0.05)
-				(type solid)
-			)
-			(layer "B.CrtYd")
-		)
-		(fp_line
-			(start -1.48 0.73)
-			(end 1.48 0.73)
-			(stroke
-				(width 0.05)
-				(type solid)
-			)
-			(layer "B.CrtYd")
-		)
-		(fp_line
-			(start -1.48 -0.73)
-			(end -1.48 0.73)
-			(stroke
-				(width 0.05)
-				(type solid)
-			)
-			(layer "B.CrtYd")
+			(start -0.8 -0.4)
+			(end 0.8 -0.4)
+			(stroke
+				(width 0.1)
+				(type solid)
+			)
+			(layer "B.Fab")
+		)
+		(fp_line
+			(start -0.8 0.1)
+			(end -0.8 -0.4)
+			(stroke
+				(width 0.1)
+				(type solid)
+			)
+			(layer "B.Fab")
+		)
+		(fp_line
+			(start -0.5 0.4)
+			(end -0.8 0.1)
+			(stroke
+				(width 0.1)
+				(type solid)
+			)
+			(layer "B.Fab")
+		)
+		(fp_line
+			(start 0.8 -0.4)
+			(end 0.8 0.4)
+			(stroke
+				(width 0.1)
+				(type solid)
+			)
+			(layer "B.Fab")
 		)
 		(fp_line
@@
 			(layer "B.Fab")
 		)
-		(fp_line
-			(start 0.8 -0.4)
-			(end 0.8 0.4)
-			(stroke
-				(width 0.1)
-				(type solid)
-			)
-			(layer "B.Fab")
-		)
-		(fp_line
-			(start -0.5 0.4)
-			(end -0.8 0.1)
-			(stroke
-				(width 0.1)
-				(type solid)
-			)
-			(layer "B.Fab")
-		)
-		(fp_line
-			(start -0.8 0.1)
-			(end -0.8 -0.4)
-			(stroke
-				(width 0.1)
-				(type solid)
-			)
-			(layer "B.Fab")
-		)
-		(fp_line
-			(start -0.8 -0.4)
-			(end 0.8 -0.4)
-			(stroke
-				(width 0.1)
-				(type solid)
-			)
-			(layer "B.Fab")
-		)
 		(fp_text user "${REFERENCE}"
 			(at 0 0 0)
@@
 		)
 		(pad "1" smd roundrect
-			(at -0.7875 0 180)
+			(at -0.7875 0)
+			(size 0.875 0.95)
+			(layers "B.Cu" "B.Mask" "B.Paste")
+			(roundrect_rratio 0.25)
+			(net 61 "GND")
+		)
+		(pad "2" smd roundrect
+			(at 0.7875 0)
 			(size 0.875 0.95)
 			(layers "B.Cu" "B.Mask" "B.Paste")
 			(roundrect_rratio 0.25)
 			(net 181 "LED_LOOP")
-		)
-		(pad "2" smd roundrect
-			(at 0.7875 0 180)
-			(size 0.875 0.95)
-			(layers "B.Cu" "B.Mask" "B.Paste")
-			(roundrect_rratio 0.25)
-			(net 61 "GND")
 		)
 		(embedded_fonts no)
@@
 			)
 		)
-		(property "Value" "R_LED"
+		(property "Value" "330 ohm"
 			(at 0 -1.43 0)
 			(layer "B.Fab")
@@
 	)
 	(gr_line
-		(start 157.734 128.016)
-		(end 154.432 128.016)
-		(stroke
-			(width 0.2)
-			(type default)
-		)
-		(locked yes)
-		(layer "B.Cu")
-		(net 61)
-	)
-	(gr_line
 		(start 150.114 106.172)
 		(end 152.146 106.172)
@@
 	)
 	(gr_line
-		(start 157.48 128.27)
+		(start 154.432 128.016)
 		(end 157.734 128.016)
 		(stroke

Commit message: PCB Fixed
Parts:
- removed J6: GPIO PINS, Connector_PinHeader_2.54mm:PinHeader_2x20_P2.54mm_Vertical
- removed REF**: LED_P, LED_SMD:LED_0603_1608Metric
- removed REF**: 330 ohm, Resistor_SMD:R_0603_1608Metric
- added C1: 470uF, Capacitor_SMD:CP_Elec_8x10, F.Cu at (111.0, 111.8)
- added C2: 10uF, Capacitor_SMD:C_0805_2012Metric, F.Cu at (115.1, 77.5)
- added C3: 0.1uF, Capacitor_SMD:C_0805_2012Metric, F.Cu at (115.2, 82.3)
- added C4: 0.1uF, Capacitor_SMD:C_0805_2012Metric, B.Cu at (155.9, 69.1)
- added C5: 0.1uF, Capacitor_SMD:C_0805_2012Metric, B.Cu at (159.8, 72.9)
- added C6: 0.1uF, Capacitor_SMD:C_0805_2012Metric, B.Cu at (155.2, 103.6)
- added C7: 0.1uF, Capacitor_SMD:C_0805_2012Metric, B.Cu at (160.1, 107.4)
- added C8: 0.1uF, Capacitor_SMD:C_0805_2012Metric, B.Cu at (155.0, 112.0)
- added D1: LED, LED_SMD:LED_0603_1608Metric, B.Cu at (130.2, 125.8)
- added D2: D_TVS, Diode_SMD:D_SMA, F.Cu at (108.7, 82.8)
- added F1: Polyfuse, Fuse:Fuse_1812_4532Metric, F.Cu at (106.4, 103.6)
- added F2: Polyfuse, Fuse:Fuse_1812_4532Metric, F.Cu at (127.8, 63.8)
- added J7: RJ45_Amphenol_RJMG1BD3B8K1ANR, Connector_RJ:RJ45_Amphenol_RJMG1BD3B8K1ANR, F.Cu at (168.2, 94.3)
- added R3: 330 ohm, Resistor_SMD:R_0805_2012Metric, B.Cu at (124.1, 126.0)
- added R4: 47k ohm, Resistor_SMD:R_0805_2012Metric, F.Cu at (145.6, 60.2)
- added U1: USBLC, Package_TO_SOT_SMD:SOT-23-6, F.Cu at (155.6, 111.4)
- added U2: USBLC, Package_TO_SOT_SMD:SOT-23-6, F.Cu at (129.4, 69.0)
- added U3: USBLC, Package_TO_SOT_SMD:SOT-23-6, F.Cu at (134.6, 69.0)
- added U4: USBLC, Package_TO_SOT_SMD:SOT-23-6, F.Cu at (139.7, 69.2)
- added U5: USBLC, Package_TO_SOT_SMD:SOT-23-6, F.Cu at (144.5, 69.2)
- added U6: TPD, Package_SON:USON-10_2.5x1.0mm_P0.5mm, F.Cu at (172.0, 117.7)
- added U7: TPS, Package_TO_SOT_SMD:SOT-23-5, F.Cu at (172.1, 111.2)
- added U8: USBLC, Package_TO_SOT_SMD:SOT-23-6, F.Cu at (154.9, 129.4)
- J3: value RJ45_LED -> GPIO Pins; footprint Connector_RJ:RJ45_Molex_0855135013_Vertical -> Connector_PinHeader_2.54mm:PinHeader_1x05_P2.54mm_Vertical
- R1, R2: value 5100 ohm -> 5.1k
- moved J5 67.9 mm to (137.5, 63.7)
- moved J2 67.8 mm to (142.5, 131.3)
- moved R1 46.4 mm to (104.3, 98.3)
- moved J4 45.2 mm to (106.6, 91.0), turned to 90 degrees
- moved R2 45.1 mm to (108.7, 98.3)
- moved J1 36.8 mm to (158.0, 121.1)
- moved J3 7.41 mm to (176.8, 104.9), turned to 180 degrees
- moved Module1 1.03 mm to (149.1, 119.9)
Connections:
- net Net-(J1-SSRX-) renamed /SSRX-
- J1 pad 1: /+5V -> Net-(J1-VBUS)
- J3 pad 1: Net-(Module1A-Ethernet_Pair1_P) -> /+3.3V
- J3 pad 2: Net-(Module1A-Ethernet_Pair1_N) -> /GPIO2
- J3 pad 3: Net-(Module1A-Ethernet_Pair0_N) -> /GPIO3
- J3 pad 4: Net-(Module1A-Ethernet_Pair2_N) -> GND
- J3 pad 5: Net-(Module1A-Ethernet_Pair2_P) -> +5V
- J4 pad A9: /+5V -> /VBUS_IN
- J4 pad B9: /+5V -> /VBUS_IN
- J5 pad 19: /+5V -> Net-(J5-+5V)
- Module1 pad 10: Net-(Module1A-Ethernet_Pair0_N) -> /Ethernet_Pair0_N
- Module1 pad 11: Net-(Module1A-Ethernet_Pair2_P) -> unconnected-(Module1A-Ethernet_Pair2_P-Pad11)
- Module1 pad 111: unconnected-(Module1B-VBUS_EN-Pad111) -> /VBUS_EN
- Module1 pad 12: Net-(Module1A-Ethernet_Pair0_P) -> /Ethernet_Pair0_P
- Module1 pad 130: Net-(J1-SSRX+) -> /SSRX+
- Module1 pad 140: Net-(J1-SSTX-) -> /SSTX-
- Module1 pad 142: Net-(J1-SSTX+) -> /SSTX+
- Module1 pad 3: Net-(Module1A-Ethernet_Pair3_P) -> unconnected-(Module1A-Ethernet_Pair3_P-Pad3)
- Module1 pad 4: Net-(Module1A-Ethernet_Pair1_P) -> /Ethernet_Pair1_P
- Module1 pad 5: Net-(Module1A-Ethernet_Pair3_N) -> unconnected-(Module1A-Ethernet_Pair3_N-Pad5)
- Module1 pad 6: Net-(Module1A-Ethernet_Pair1_N) -> /Ethernet_Pair1_N
- Module1 pad 77: /+5V -> +5V
- Module1 pad 79: /+5V -> +5V
- Module1 pad 81: /+5V -> +5V
- Module1 pad 83: /+5V -> +5V
- Module1 pad 85: /+5V -> +5V
- Module1 pad 87: /+5V -> +5V
- Module1 pad 9: Net-(Module1A-Ethernet_Pair2_N) -> unconnected-(Module1A-Ethernet_Pair2_N-Pad9)
Routing:
- net /SSRX+: track 0.00 -> 116.8 mm, vias 0 -> 1
- net /SSTX-: track 0.00 -> 102.8 mm, vias 0 -> 1
- net /SSTX+: track 0.00 -> 99.0 mm, vias 0 -> 1
- net GND: track 287.1 -> 195.2 mm, vias 69 -> 81
- net /VBUS_EN: track 0.00 -> 68.3 mm, vias 0 -> 1
- net /SSRX-: track 78.8 -> 145.4 mm, vias 2 -> 1
- net +5V: track 0.00 -> 65.6 mm, vias 0 -> 19
- net /HDMI0_TX0_N: track 46.9 -> 108.2 mm, vias 1 -> 3
- net Net-(Module1A-Ethernet_Pair0_N): track 46.9 -> 0.00 mm, vias 2 -> 0
- net /HDMI0_SDA: track 45.3 -> 90.8 mm
- net Net-(Module1A-Ethernet_Pair0_P): track 44.5 -> 0.00 mm, vias 1 -> 0
- net /+5V: track 36.4 -> 0.00 mm, vias 5 -> 0
- net Net-(Module1A-Ethernet_Pair1_N): track 36.3 -> 0.00 mm, vias 1 -> 0
- net Net-(Module1A-Ethernet_Pair1_P): track 35.0 -> 0.00 mm, vias 1 -> 0
- net /HDMI0_TX2_N: track 49.9 -> 84.4 mm
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- added copper zone on B.Cu, net +5V
- added copper zone on In3.Cu, net +5V
- added copper zone on B.Cu, net GND
- added copper zone on F.Cu, net GND
- removed copper zone on In3.Cu, net /+5V

Commit message: Reduced to 6 layers
Parts:
- moved J5 3.28 mm to (137.9, 60.5), turned to 180 degrees
Routing:
- net /HDMI0_TX0_N: track 108.2 -> 61.7 mm, vias 3 -> 1
- net /SSRX-: track 145.4 -> 108.6 mm
- net /HDMI0_SDA: track 90.8 -> 55.6 mm, vias 1 -> 2
- net /HDMI0_TX0_P: track 78.8 -> 113.9 mm, vias 1 -> 2
- net /SSRX+: track 116.8 -> 84.3 mm
- net GND: track 195.2 -> 226.4 mm, vias 81 -> 72
- net /HDMI0_TX2_N: track 84.4 -> 102.3 mm, vias 1 -> 3
- net /HDMI0_TX2_P: track 80.3 -> 63.8 mm, vias 1 -> 3
- net /SSTX-: track 102.8 -> 87.5 mm
- net /MIPI0_C_P: track 48.9 -> 61.6 mm
- net /SSTX+: track 99.0 -> 87.0 mm
- net /GPIO2: track 33.1 -> 41.8 mm, vias 1 -> 0
- net /HDMI0_CLK_N: track 64.0 -> 72.0 mm
- net /HDMI0_CLK_P: track 65.0 -> 73.0 mm
- net /GPIO3: track 30.5 -> 38.0 mm
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- removed copper zone on In6.Cu, net GND
Other:
- copper layers 8 -> 6
